Commit message: stage robots test was success but needs backward move and route error bugs fix

File: robot/ws/src/trp1_description/urdf/trp1.xacro (robot description, xacro)
@@ -96,4 +96,10 @@
     -->
   </link>
+  <link name="imu_link"/>
+  <joint type="fixed" name="imu_joint">
+    <origin xyz="0 0 0.18" rpy="0 0 0"/>
+    <parent link="base_link"/>
+    <child link="imu_link"/>
+  </joint>
   <!-- Intel D430 -->
   <joint type="fixed" name="camera_joint">

File: robot/ws/src/trp1_description/urdf/trp1_stage.urdf.xacro (robot description, xacro)
@@ -97,4 +97,10 @@
     -->
   </link>
+  <link name="imu_link"/>
+  <joint type="fixed" name="imu_joint">
+    <origin xyz="0 0 0.18" rpy="0 0 0"/>
+    <parent link="base_link"/>
+    <child link="imu_link"/>
+  </joint>
   <!-- Центральный laser убран.
        Его TF и положение оставляет stage_ros2: base_link -> laser -->
